Commit message: Refactoring so it makes more sense

File: src/so_arm100/urdf/so_arm100.urdf (robot description, URDF)
Before this commit: robot st3215_ros2_control, 8 links, 7 joints
Links:
- link Base: geometry collision mesh filename=package://so_arm100/meshes/Base.STL; visual mesh filename=package://so_arm100/meshes/Base.STL
- link Fixed_Jaw: geometry collision mesh filename=package://so_arm100/meshes/Fixed_Jaw.STL; visual mesh filename=package://so_arm100/meshes/Fixed_Jaw.STL
- link Lower_Arm: geometry collision mesh filename=package://so_arm100/meshes/Lower_Arm.STL; visual mesh filename=package://so_arm100/meshes/Lower_Arm.STL
- link Moving_Jaw: geometry collision mesh filename=package://so_arm100/meshes/Moving_Jaw.STL; visual mesh filename=package://so_arm100/meshes/Moving_Jaw.STL
- link Rotation_Pitch: geometry collision mesh filename=package://so_arm100/meshes/Rotation_Pitch.STL; visual mesh filename=package://so_arm100/meshes/Rotation_Pitch.STL
- link Upper_Arm: geometry collision mesh filename=package://so_arm100/meshes/Upper_Arm.STL; visual mesh filename=package://so_arm100/meshes/Upper_Arm.STL
- link Wrist_Pitch_Roll: geometry collision mesh filename=package://so_arm100/meshes/Wrist_Pitch_Roll.STL; visual mesh filename=package://so_arm100/meshes/Wrist_Pitch_Roll.STL
Joints:
- joint Wrist_Pitch: limit lower=-1.5708 upper=1.5708 effort=3 velocity=2 -> lower=-2.5708 upper=0.2 effort=3 velocity=2
- joint Wrist_Roll: limit lower=-3.14 upper=3.14 effort=3 velocity=2 -> lower=-0.5 upper=3.14 effort=3 velocity=2

File: src/so_arm100_moveit/config/so_arm100.ros2_control.xacro (robot description, xacro)
@@ -1,5 +1,5 @@
 <?xml version="1.0"?>
 <robot xmlns:xacro="http://www.ros.org/wiki/xacro">
-    <xacro:macro name="st3215_ros2_control_ros2_control" params="name initial_positions_file">
+    <xacro:macro name="so_arm100_ros2_control" params="name initial_positions_file">
         <xacro:property name="initial_positions" value="${load_yaml(initial_positions_file)['initial_positions']}"/>
         <ros2_control name="${name}" type="system">
